File: picoSYS/picoSYS/picoSYS.kicad_sch (KiCad schematic)
At the start: 0 parts

Commit message: reading info
Parts:
- added A1: RaspberryPi_Pico, Module_RaspberryPi_Pico:RaspberryPi_Pico_Common, symbol MCU_Module_RaspberryPi_Pico:RaspberryPi_Pico
- added A2: RaspberryPi_Pico_W, Module_RaspberryPi_Pico:RaspberryPi_Pico_Common, symbol MCU_Module_RaspberryPi_Pico:RaspberryPi_Pico_W
- added C8: 330uF 6.3V, symbol Device:C_Polarized
- added D2: 5V, symbol Device:D_Zener
- added F1: 500mA, symbol Device:Polyfuse_Small
- added Q1: BD237, Package_TO_SOT_THT:TO-126-3_Vertical, symbol Transistor_BJT:BD237
- added R10, R11, R37, R38, R39, R4, R40, R41, R42, R43, R44, R5, R6, R7, R8, R9: 2.2k, symbol Device:R
- added R12, R23, R24, R26, R27, R28: 10kR, symbol Device:R
- added R13, R14, R15, R16, R17, R18, R19, R20, R29, R30, R31, R32, R33, R34, R35, R36, R45: 1k, symbol Device:R
- added R21, R47: 100kR, symbol Device:R
- added R22: 27kR, symbol Device:R
- added R25: 1kR, symbol Device:R
- added R46: 10R, symbol Device:R
- added R48: 47kR, symbol Device:R
- added U2, U3: NE5532, symbol Amplifier_Operational:NE5532
Connections:
- new net: R16.1, R17.2, R8.1
- new net: A1.10 (GPIO7), R8.2
- new net: R15.1, R16.2, R7.1
- new net: R14.1, R15.2, R6.1
- new net: R36.1, R44.1, R47.1
- new net: R47.2, R48.1, U3.5 (+)
- new net: A1.15 (GPIO11), R12.2
- new net: R27.2, R28.1, U3.2 (-)
- new net: R23.1, R26.1, U3.3 (+)
- new net: R24.1, R25.1, U2.5 (+)
- new net: R10.1, R18.1, R19.2
- new net: A1.12 (GPIO9), R10.2
- new net: R34.1, R35.2, R42.1
- new net: R33.1, R34.2, R41.1
- new net: A1.7 (GPIO5), R6.2
- new net: R31.1, R32.2, R39.1
- new net: A2.4 (GPIO2), R39.2
- new net: A1.9 (GPIO6), R7.2
- new net: R26.2, U2.6 (-), U2.7
- new net: Q1.1 (E), R46.1, U3.6 (-)
- new net: R45.1, U3.7
- new net: R13.1, R14.2, R5.1
- new net: R13.2, R20.1, R4.1
- new net: R21.2, R22.2, U2.3 (+)
- new net: A2.6 (GPIO4), R41.2
- new net: R32.1, R33.2, R40.1
- new net: R17.1, R18.2, R9.1
- new net: A1.11 (GPIO8), R9.2
- new net: A1.5 (GPIO3), R4.2
- new net: A1.14 (GPIO10), R11.2
- new net: A1.6 (GPIO4), R5.2
- new net: R29.1, R30.2, R37.1
- new net: A2.5 (GPIO3), R40.2
- new net: R23.2, U2.1, U2.2 (-)
- new net: A2.7 (GPIO5), R42.2
- new net: A2.1 (GPIO0), R37.2
- new net: R35.1, R36.2, R43.1
- new net: A2.9 (GPIO6), R43.2
- new net: Q1.3 (B), R45.2
- new net: R30.1, R31.2, R38.1
- new net: A2.10 (GPIO7), R44.2
- new net: A2.2 (GPIO1), R38.2
- new net +5V: F1.1
- new net -2V: U2.4 (V-), U3.4 (V-)
- new net 5v: A1.39 (VSYS), A2.40 (VBUS), C8.1, D2.1 (K), F1.2, Q1.2 (C), U2.8 (V+), U3.8 (V+)
- new net AUDIO_OUT: R46.2
- new net GND: A1.13 (GND), A1.18 (GND), A1.23 (GND), A1.28 (GND), A1.3 (GND), A1.38 (GND), A1.8 (GND), A2.13 (GND), A2.18 (GND), A2.23 (GND), A2.28 (GND), A2.3 (GND), A2.38 (GND), A2.8 (GND), C8.2, D2.2 (A), R20.2, R22.1, R25.2, R28.2, R29.2, R48.2
- new net VIDEO_DAC: R11.1, R19.1, R21.1
- new net VIDEO_OUT: R27.1, U3.1
- new net ~{SYNC}: R12.1, R24.2

Commit message: working audio test
Parts:
- removed R46: 10R, symbol Device:R
- R29, R30, R31, R32, R33, R34, R35, R36: value 1k -> 330R
- R37, R38, R39, R40, R41, R42, R43, R44: value 2.2k -> 680R
- R47: value 100kR -> 10kR
- R48: value 47kR -> 6.8kR
Connections:
- net AUDIO_OUT: now also Q1.1 (E), U3.6 (-)

Commit message: updated schematic to better reflect real hardware, removed a debug message
Parts:
- removed R12: 10kR, symbol Device:R
- added C1, C10, C3, C4, C9: 1uF, symbol Device:C
- added C2: 6x 330uF 6.3V, symbol Device:C_Polarized
- added U4: ICL7660, symbol Regulator_SwitchedCapacitor:ICL7660
- added U5: L78L33_TO92, Package_TO_SOT_THT:TO-92_Inline, symbol Regulator_Linear:L78L33_TO92
- R21: value 100kR -> 10kR
- R22: value 27kR -> 2.7kR
- U2, U3: value NE5532 -> OPA1612AxD; symbol Amplifier_Operational:NE5532 -> Amplifier_Operational:OPA1612AxD
Connections:
- net 5v: now also C10.1, U5.3 (VI); no longer U2.8 (V+), U3.8 (V+)
- net GND: now also C10.2, C2.2, C9.2, U4.3 (GND), U5.2 (GND)
- net ~{SYNC}: now also A1.15 (GPIO11)
- net SDA: now reaches A1.21 (GPIO16)
- net SDA: now also A2.21 (GPIO16)
- net SCL: now reaches A1.22 (GPIO17)
- net SCL: now also A2.22 (GPIO17)
- net -2V renamed -3.3V
- net -3.3V: now also C2.1, C3.2, C4.2, U4.5 (VOUT)
- new net: C1.1, U4.2 (CAP+)
- new net: C1.2, U4.4 (CAP-)
- new net +3.3V: C3.1, C4.1, C9.1, U2.8 (V+), U3.8 (V+), U4.8 (V+), U5.1 (VO)
Other:
- removed sheet inverting_supply
- moved on the sheet: U2C, U3C
